Commit message: robot_description V0.1.0

File: robot_description/urdf/BGK_robot.urdf.xacro (robot description, xacro)
@@ -1,4 +1,4 @@
 <?xml version="1.0"?>
-<robot name="bumperbot" xmlns:xacro="http://ros.org/wiki/xacro">
+<robot name="BGK_bot" xmlns:xacro="http://ros.org/wiki/xacro">
     <link name="base_footprint"/>
     <link name="base_link">
@@ -7,5 +7,4 @@
             <geometry>
                 <box size="0.15 0.1 0.05"/>
-                <!-- <cylinder length="0.1" radius="0.2" /> -->
             </geometry>
         </collision>
@@ -27,5 +26,4 @@
         <origin xyz="0 0 0" rpy="1.57 0 0" />
         <geometry>
-            <!-- <cylinder length="0.007" radius="0.03" /> -->
             <mesh filename="package://robot_description/meshes/wheel_right_link.STL" />
         </geometry>
@@ -34,5 +32,4 @@
             <origin xyz="0 0 0" rpy="1.57 0 0" />
             <geometry>
-                <!-- <sphere radius="0.033"/> -->
                 <cylinder length="0.007" radius="0.03" />
             </geometry>
@@ -49,5 +46,4 @@
             <origin xyz="0 0 0" rpy="-1.57 0 0" />
             <geometry>
-                <!-- <cylinder length="0.007" radius="0.03" /> -->
                 <mesh filename="package://robot_description/meshes/wheel_left_link.STL" />
             </geometry>
@@ -56,5 +52,4 @@
             <origin xyz="0 0 0" rpy="-1.57 0 0" />
             <geometry>
-                <!-- <sphere radius="0.033"/> -->
                 <cylinder length="0.007" radius="0.03" />
             </geometry>

Commit message: update code

File: robot_description/urdf/BGK_robot.urdf.xacro (robot description, xacro)
@@ -1,5 +1,5 @@
 <?xml version="1.0"?>
 <robot name="BGK_bot" xmlns:xacro="http://ros.org/wiki/xacro">
-    <link name="base_footprint"/>
+    <link name="odom"/>
     <link name="base_link">
         <collision>
@@ -18,5 +18,5 @@
     </link>
     <joint name="base_joint" type="fixed">
-        <parent link="base_footprint"/>
+        <parent link="odom"/>
         <child link="base_link" />
         <origin xyz="0 0 0.033" rpy="0 0 0"/>
